Commit message: Spawned BOT without Plugins

File: mr_robot_description/urdf/mr_robot.xacro (robot description, xacro)
@@ -13,5 +13,5 @@
     <origin xyz="0 0 0" rpy="0 0 0"/>
     <geometry>
-      <mesh filename="package://mr_robot_description/meshes/base_link.stl" scale="0.001 0.001 0.001"/>
+      <mesh filename="file://$(find mr_robot_description)/meshes/base_link.stl" scale="0.001 0.001 0.001"/>
     </geometry>
     <material name="silver"/>
@@ -20,5 +20,5 @@
     <origin xyz="0 0 0" rpy="0 0 0"/>
     <geometry>
-      <mesh filename="package://mr_robot_description/meshes/base_link.stl" scale="0.001 0.001 0.001"/>
+      <mesh filename="file://$(find mr_robot_description)/meshes/base_link.stl" scale="0.001 0.001 0.001"/>
     </geometry>
   </collision>
@@ -33,5 +33,5 @@
     <origin xyz="0.0 0.0 0.0035" rpy="0 0 0"/>
     <geometry>
-      <mesh filename="package://mr_robot_description/meshes/lidar_1_1_1_1.stl" scale="0.001 0.001 0.001"/>
+      <mesh filename="file://$(find mr_robot_description)/meshes/lidar_1_1_1_1.stl" scale="0.001 0.001 0.001"/>
     </geometry>
     <material name="silver"/>
@@ -40,5 +40,5 @@
     <origin xyz="0.0 0.0 0.0035" rpy="0 0 0"/>
     <geometry>
-      <mesh filename="package://mr_robot_description/meshes/lidar_1_1_1_1.stl" scale="0.001 0.001 0.001"/>
+      <mesh filename="file://$(find mr_robot_description)/meshes/lidar_1_1_1_1.stl" scale="0.001 0.001 0.001"/>
     </geometry>
   </collision>
@@ -53,5 +53,5 @@
     <origin xyz="0.40035 -0.190925 0.0556" rpy="0 0 0"/>
     <geometry>
-      <mesh filename="package://mr_robot_description/meshes/right_wheel_1_1_1_1.stl" scale="0.001 0.001 0.001"/>
+      <mesh filename="file://$(find mr_robot_description)/meshes/right_wheel_1_1_1_1.stl" scale="0.001 0.001 0.001"/>
     </geometry>
     <material name="silver"/>
@@ -60,5 +60,5 @@
     <origin xyz="0.40035 -0.190925 0.0556" rpy="0 0 0"/>
     <geometry>
-      <mesh filename="package://mr_robot_description/meshes/right_wheel_1_1_1_1.stl" scale="0.001 0.001 0.001"/>
+      <mesh filename="file://$(find mr_robot_description)/meshes/right_wheel_1_1_1_1.stl" scale="0.001 0.001 0.001"/>
     </geometry>
   </collision>
@@ -73,5 +73,5 @@
     <origin xyz="0.39965 0.182675 0.0556" rpy="0 0 0"/>
     <geometry>
-      <mesh filename="package://mr_robot_description/meshes/left_wheel_1_1_1_1.stl" scale="0.001 0.001 0.001"/>
+      <mesh filename="file://$(find mr_robot_description)/meshes/left_wheel_1_1_1_1.stl" scale="0.001 0.001 0.001"/>
     </geometry>
     <material name="silver"/>
@@ -80,5 +80,5 @@
     <origin xyz="0.39965 0.182675 0.0556" rpy="0 0 0"/>
     <geometry>
-      <mesh filename="package://mr_robot_description/meshes/left_wheel_1_1_1_1.stl" scale="0.001 0.001 0.001"/>
+      <mesh filename="file://$(find mr_robot_description)/meshes/left_wheel_1_1_1_1.stl" scale="0.001 0.001 0.001"/>
     </geometry>
   </collision>
